Commit message: Controller fungerer på ny bil. trenger sensorer

File: urdf/ack.xacro (robot description, xacro)
@@ -1,9 +1,13 @@
 <?xml version="1.0" ?>
 <robot name="ack" xmlns:xacro="http://ros.org/wiki/xacro">
-    <!-- 瀹氫箟榛戣壊鏉愯川 -->
+  <!-- Parameters -->
+   <xacro:property name="M_PI" value="3.14159265359"/>
+   <xacro:property name="max_steering_angle" value="0.5"/> <!-- 28.65 grader -->
+   <xacro:property name="max_velocity" value="0.6"/>
+   <xacro:property name="max_wheel_angular_velocity" value="${2 * max_velocity/0.067}"/> <!-- Wheel diameter = 0.067 -->
   <material name="black">
     <color rgba="0 0 0 1"/>
   </material>
-  <!-- 瀹氫箟 base_link -->
+  <!-- base_link -->
   <link name="base_link">
     <inertial>
@@ -28,7 +32,7 @@
     </collision>
   </link>
-  <!-- 娣诲姞 base_footprint 閾炬帴 -->
+  <!-- base_footprint -->
   <link name="base_footprint"/>
-  <!-- 瀹氫箟 base_footprint 鍒?base_link 鐨勫浐瀹氬叧鑺?-->
+  <!-- base_footprint to base_link -->
   <joint name="base_footprint_to_base_link" type="fixed">
     <parent link="base_footprint"/>
@@ -36,5 +40,5 @@
     <origin xyz="0 0 0.07" rpy="0 0 0"/>
   </joint>
-  <!-- 瀹氫箟鍏朵粬閾炬帴鍜屽叧鑺?-->
+  <!-- Wheel links-->
   <link name="wheel_lf_Link">
     <inertial>
@@ -63,5 +67,5 @@
     <parent link="base_link"/>
     <child link="wheel_lf_Link"/>
-    <axis xyz="-2.2918E-05 1 1.9551E-05"/>
+    <axis xyz="-2.2918E-05 1.9551E-05 1"/>
   </joint>
   <link name="wheel_rf_Link">
@@ -91,5 +95,5 @@
     <parent link="base_link"/>
     <child link="wheel_rf_Link"/>
-    <axis xyz="-2.2918E-05 1 1.9551E-05"/>
+    <axis xyz="-2.2918E-05 1.9551E-05 1"/>
   </joint>
   <link name="wheel_lb_Link">
@@ -178,3 +182,57 @@
   </joint>
   <xacro:include filename="$(find rc_gazebo)/urdf/imu.urdf.xacro"/>
+  <!-- Gazebo Control -->
+  <ros2_control name="ack_control" type="system">
+    <hardware>
+      <plugin>gz_ros2_control/GazeboSimSystem</plugin>
+    </hardware>
+    <!-- Front wheels (steering joints) -->
+    <joint name="wheel_lf_Joint">
+      <command_interface name="position">
+        <param name="min">${-max_steering_angle}</param>
+        <param name="max">${max_steering_angle}</param>
+      </command_interface>
+      <state_interface name="position"/>
+      <state_interface name="velocity"/>
+    </joint>
+    <joint name="wheel_rf_Joint">
+      <command_interface name="position">
+        <param name="min">${-max_steering_angle}</param>
+        <param name="max">${max_steering_angle}</param>
+      </command_interface>
+      <state_interface name="position"/>
+      <state_interface name="velocity"/>
+    </joint>
+    <!-- Rear wheels (drive joints) -->
+    <joint name="wheel_lb_Joint">
+      <command_interface name="velocity">
+        <param name="min">${-max_wheel_angular_velocity}</param>
+        <param name="max">${max_wheel_angular_velocity}</param>
+      </command_interface>
+      <state_interface name="position"/>
+      <state_interface name="velocity"/>
+    </joint>
+    <joint name="wheel_rb_Joint">
+      <command_interface name="velocity">
+        <param name="min">${-max_wheel_angular_velocity}</param>
+        <param name="max">${max_wheel_angular_velocity}</param>
+      </command_interface>
+      <state_interface name="position"/>
+      <state_interface name="velocity"/>
+    </joint>
+  </ros2_control>
+  <gazebo>
+    <plugin filename="gz-sim-joint-state-publisher-system"
+            name="gz::sim::systems::JointStatePublisher">
+      <topic>joint_states</topic>
+      <joint_name>wheel_lf_Joint</joint_name>
+      <joint_name>wheel_rf_Joint</joint_name>
+      <joint_name>wheel_lb_Joint</joint_name>
+      <joint_name>wheel_rb_Joint</joint_name>
+    </plugin>
+    <plugin filename="gz_ros2_control-system"
+            name="gz_ros2_control::GazeboSimROS2ControlPlugin">
+      <parameters>$(find rc_gazebo)/config/gz_ros2_control.yaml</parameters>
+    </plugin>
+  </gazebo>
 </robot>

Commit message: lidar sensor (må sjekke rpy mot ekte bil)

File: urdf/ack.xacro (robot description, xacro)
@@ -153,4 +153,10 @@
     <axis xyz="-2.2787E-05 1 1.9439E-05"/>
   </joint>
+  <joint name="lidar_Joint" type="fixed">
+    <origin rpy="0 0 0" xyz="-0.0096019 -8.533E-05 0.092501"/>
+    <parent link="base_link"/>
+    <child link="lidar_frame"/>
+    <axis xyz="0 0 0"/>
+  </joint>
   <link name="lidar_frame">
     <inertial>
@@ -175,10 +181,4 @@
     </collision>
   </link>
-  <joint name="lidar_Joint" type="fixed">
-    <origin rpy="0 0 0" xyz="-0.0096019 -8.533E-05 0.092501"/>
-    <parent link="base_link"/>
-    <child link="lidar_frame"/>
-    <axis xyz="0 0 0"/>
-  </joint>
   <xacro:include filename="$(find rc_gazebo)/urdf/imu.urdf.xacro"/>
   <!-- Gazebo Control -->
@@ -236,3 +236,39 @@
     </plugin>
   </gazebo>
+  <!-- Sensorer -->
+  <!-- <gazebo>
+    <plugin name='gz::sim::systems::Sensors' filename='gz-sim-sensors-system'>
+      <render_engine>ogre2</render_engine>
+    </plugin>
+  </gazebo> -->
+  <gazebo reference="lidar_frame">
+    <sensor name="lidar_sensor" type="gpu_lidar">
+      <always_on>true</always_on>
+      <update_rate>10</update_rate>
+      <visualize>true</visualize>
+      <topic>/sensors/lidar/raw</topic>
+      <enable_metrics>false</enable_metrics>
+      <pose relative_to="lidar_frame"> 0 0 0 0 0 3.14159265359 </pose>
+      <lidar>
+        <scan>
+          <horizontal>
+            <samples>450</samples>
+            <resolution>1</resolution>
+            <min_angle>-3.14159265359</min_angle>
+            <max_angle>3.14159265359</max_angle>
+          </horizontal>
+        </scan>
+        <range>
+          <min>0.05</min>
+          <max>20</max>
+          <resolution>0.01</resolution>
+        </range>
+        <noise>
+          <type>gaussian</type>
+          <mean>0</mean>
+          <stddev>0</stddev>
+        </noise>
+      </lidar>
+    </sensor>
+  </gazebo>
 </robot>

Commit message: lidar i egen fil

File: urdf/ack.xacro (robot description, xacro)
@@ -1,4 +1,5 @@
 <?xml version="1.0" ?>
 <robot name="ack" xmlns:xacro="http://ros.org/wiki/xacro">
+  <xacro:include filename="$(find rc_gazebo)/urdf/lidar.xacro" />
   <!-- Parameters -->
    <xacro:property name="M_PI" value="3.14159265359"/>
@@ -153,32 +154,4 @@
     <axis xyz="-2.2787E-05 1 1.9439E-05"/>
   </joint>
-  <joint name="lidar_Joint" type="fixed">
-    <origin rpy="0 0 0" xyz="-0.0096019 -8.533E-05 0.092501"/>
-    <parent link="base_link"/>
-    <child link="lidar_frame"/>
-    <axis xyz="0 0 0"/>
-  </joint>
-  <link name="lidar_frame">
-    <inertial>
-      <origin rpy="0 0 0" xyz="8.65086433231368E-05 9.02624784523964E-05 -0.0183546134614858"/>
-      <mass value="0.0405423044068563"/>
-      <inertia ixx="4.98470776877503E-06" ixy="-1.54076264166869E-07" ixz="2.05182706824286E-09" iyy="5.03926730822203E-06" iyz="1.1006285118993E-08" izz="8.25645669548359E-06"/>
-    </inertial>
-    <visual>
-      <origin rpy="0 0 0" xyz="0 0 0"/>
-      <geometry>
-        <mesh filename="models://acker/lidar_Link.STL"/>
-      </geometry>
-      <material name="">
-        <color rgba="0.1 0.1 0.1 1"/>
-      </material>
-    </visual>
-    <collision>
-      <origin rpy="0 0 0" xyz="0 0 0"/>
-      <geometry>
-        <mesh filename="models://acker/lidar_Link.STL"/>
-      </geometry>
-    </collision>
-  </link>
   <xacro:include filename="$(find rc_gazebo)/urdf/imu.urdf.xacro"/>
   <!-- Gazebo Control -->
@@ -237,38 +210,4 @@
   </gazebo>
   <!-- Sensorer -->
-  <!-- <gazebo>
-    <plugin name='gz::sim::systems::Sensors' filename='gz-sim-sensors-system'>
-      <render_engine>ogre2</render_engine>
-    </plugin>
-  </gazebo> -->
-  <gazebo reference="lidar_frame">
-    <sensor name="lidar_sensor" type="gpu_lidar">
-      <always_on>true</always_on>
-      <update_rate>10</update_rate>
-      <visualize>true</visualize>
-      <topic>/sensors/lidar/raw</topic>
-      <enable_metrics>false</enable_metrics>
-      <pose relative_to="lidar_frame"> 0 0 0 0 0 3.14159265359 </pose>
-      <lidar>
-        <scan>
-          <horizontal>
-            <samples>450</samples>
-            <resolution>1</resolution>
-            <min_angle>-3.14159265359</min_angle>
-            <max_angle>3.14159265359</max_angle>
-          </horizontal>
-        </scan>
-        <range>
-          <min>0.05</min>
-          <max>20</max>
-          <resolution>0.01</resolution>
-        </range>
-        <noise>
-          <type>gaussian</type>
-          <mean>0</mean>
-          <stddev>0</stddev>
-        </noise>
-      </lidar>
-    </sensor>
-  </gazebo>
+  <xacro:lidar_sensor></xacro:lidar_sensor>
 </robot>

Commit message: topic og link navn

File: urdf/ack.xacro (robot description, xacro)
@@ -34,12 +34,4 @@
     </collision>
   </link>
-  <!-- base_footprint -->
-  <link name="base_footprint"/>
-  <!-- base_footprint to base_link -->
-  <joint name="base_footprint_to_base_link" type="fixed">
-    <parent link="base_footprint"/>
-    <child link="base_link"/>
-    <origin xyz="0 0 0.07" rpy="0 0 0"/>
-  </joint>
   <!-- Wheel links-->
   <link name="wheel_lf_Link">

File: urdf/lidar.xacro (robot description, xacro)
@@ -6,8 +6,8 @@
             <origin rpy="0 0 0" xyz="-0.0096019 -8.533E-05 0.092501"/>
             <parent link="base_link"/>
-            <child link="lidar_frame"/>
+            <child link="lidar_link"/>
             <axis xyz="0 0 0"/>
         </joint>
-        <link name="lidar_frame">
+        <link name="lidar_link">
             <inertial>
                 <origin rpy="0 0 0" xyz="8.65086433231368E-05 9.02624784523964E-05 -0.0183546134614858"/>
@@ -32,6 +32,7 @@
         </link>
         <!-- Faktiske sensoren -->
-        <gazebo reference="lidar_frame">
+        <gazebo reference="lidar_link">
             <sensor name="lidar_sensor" type="gpu_lidar">
+                <gz_frame_id>lidar_link</gz_frame_id>
                 <always_on>true</always_on>
                 <update_rate>10</update_rate>
@@ -39,5 +40,5 @@
                 <topic>/sensors/lidar/scan_raw</topic>
                 <enable_metrics>false</enable_metrics>
-                <pose relative_to="lidar_frame"> 0 0 0 0 0 3.14159265359 </pose>
+                <pose relative_to="lidar_link"> 0 0 0 0 0 3.14159265359 </pose>
                 <lidar>
                     <scan>
