Commit message: gjorde imu til 0 rotation for nå

File: urdf/imu.xacro (robot description, xacro)
@@ -6,5 +6,6 @@
         </link>
         <joint name="imu_joint" type="fixed">
-            <origin xyz="0 0 ${0.025 - 0.0295 + 0.0965/2 + 0.0678410821576746}" rpy="0 0 ${-M_PI/2}" />
+            <origin xyz="0 0 ${0.025 - 0.0295 + 0.0965/2 + 0.0678410821576746}" rpy="0 0 0" />
+            <!-- <origin xyz="0 0 ${0.025 - 0.0295 + 0.0965/2 + 0.0678410821576746}" rpy="0 0 ${-M_PI/2}" /> -->
             <parent link="base_link" />
             <child link="imu_link" />
